File: PCB - KiCad/DSKY_driver/DSKY_driver.kicad_pcb (KiCad board)
At the start: 2 copper layers, 43 x 94.3 mm, 39 parts, among them IC3 ATSAMD21E, J1 Conn_15X4, J2 Conn_15X4, J3 CUI_power_jack, J4 Conn_15X4, Q2 reset, U1 HV507, U2 LT3468, U3 AP2204K-3.3, U4 AP2204K-5.0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

Commit message: Shrink PCB outline
Parts:
- renumbered TP4 to 3V3, TP3 to GND, TP1 to SWC, TP2 to SWD
Other:
- board size 43 x 94.3 mm -> 43 x 92.3 mm
Changed lines of the file:
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@@
-(kicad_pcb (version 20171130) (host pcbnew "(5.1.0)-1")
+(kicad_pcb (version 20171130) (host pcbnew "(5.0.0)")
   (general
     (thickness 1.6)
@@
     (zone_45_only no)
     (trace_min 0.2)
+    (segment_width 0.15)
+    (edge_width 0.15)
     (via_size 0.508)
     (via_drill 0.254)
@@
     (uvia_min_size 0.2)
     (uvia_min_drill 0.1)
-    (edge_width 0.15)
-    (segment_width 0.15)
     (pcb_text_width 0.3)
     (pcb_text_size 1 1)
@@
     (tags "test point SMD pad")
     (attr virtual)
-    (fp_text reference TP1 (at 0 -1.448) (layer F.SilkS)
+    (fp_text reference SWC (at 0 -1.448) (layer F.SilkS)
       (effects (font (size 0.75 0.75) (thickness 0.1)))
     )
@@
     (tags "test point SMD pad")
     (attr virtual)
-    (fp_text reference TP2 (at -0.675 -1.35) (layer F.SilkS)
+    (fp_text reference SWD (at -0.675 -1.35) (layer F.SilkS)
       (effects (font (size 0.75 0.75) (thickness 0.1)))
     )
@@
     (tags "test point SMD pad")
     (attr virtual)
-    (fp_text reference TP3 (at 0.775 -1.55) (layer F.SilkS)
+    (fp_text reference GND (at 0.775 -1.55) (layer F.SilkS)
       (effects (font (size 0.75 0.75) (thickness 0.1)))
     )
@@
     (tags "test point SMD pad")
     (attr virtual)
-    (fp_text reference TP4 (at -0.45 -1.5) (layer F.SilkS)
+    (fp_text reference 3V3 (at -0.45 -1.5) (layer F.SilkS)
       (effects (font (size 0.75 0.75) (thickness 0.1)))
     )
@@
     (effects (font (size 1 1) (thickness 0.1)))
   )
-  (gr_text "CAUTION:  HIGH VOLTAGE" (at 139.175 130.7) (layer F.SilkS)
+  (gr_text "CAUTION:  HIGH VOLTAGE" (at 160.25 108) (layer F.SilkS)
     (effects (font (size 1 1) (thickness 0.1)))
   )
@@
   (gr_line (start 138.4 71.675) (end 138.4 73.625) (layer F.SilkS) (width 0.15))
   (gr_line (start 137.825 64.125) (end 137.825 66.075) (layer F.SilkS) (width 0.15))
-  (gr_line (start 129 132) (end 129.025 37.7) (layer Edge.Cuts) (width 0.15))
-  (gr_line (start 172 132) (end 129 132) (layer Edge.Cuts) (width 0.15))
-  (gr_line (start 171.975 37.675) (end 172 132) (layer Edge.Cuts) (width 0.15))
+  (gr_line (start 129 130) (end 129.025 37.7) (layer Edge.Cuts) (width 0.15))
+  (gr_line (start 172 130) (end 129 130) (layer Edge.Cuts) (width 0.15))
+  (gr_line (start 171.975 37.675) (end 172 130) (layer Edge.Cuts) (width 0.15))
   (gr_line (start 129.025 37.7) (end 171.975 37.675) (layer Edge.Cuts) (width 0.15))
   (gr_line (start 120.834 27.223) (end 183.27 27.223) (layer Dwgs.User) (width 0.4))
@@
     (effects (font (size 1.2065 1.2065) (thickness 0.1016)) (justify right top))
   )
-  (segment (start 158.604 115.75) (end 157.829 114.975) (width 0.2) (layer Bottom) (net 60))
-  (segment (start 158.604 117.6) (end 158.604 115.75) (width 0.2) (layer Bottom) (net 60))
-  (via (at 155.725 114.8) (size 0.508) (drill 0.254) (layers Top Bottom) (net 60))
-  (segment (start 157.829 114.975) (end 155.9 114.975) (width 0.2) (layer Bottom) (net 60))
-  (segment (start 155.9 114.975) (end 155.725 114.8) (width 0.2) (layer Bottom) (net 60))
-  (segment (start 157.875 124.925) (end 156.65 124.925) (width 0.2) (layer Bottom) (net 95))
-  (segment (start 158.604 122.4) (end 158.604 124.196) (width 0.2) (layer Bottom) (net 95))
-  (segment (start 158.604 124.196) (end 157.875 124.925) (width 0.2) (layer Bottom) (net 95))
   (via (at 138.55 75.325) (size 0.508) (drill 0.254) (layers Top Bottom) (net 1))
   (segment (start 138.55 75.325) (end 141.625 75.325) (width 0.4) (layer Top) (net 1))
@@
   (segment (start 156.5 110.6) (end 156.4 110.5) (width 0.2) (layer Top) (net 59))
   (segment (start 156.5 114.15) (end 156.5 110.6) (width 0.2) (layer Top) (net 59))
+  (segment (start 158.604 115.75) (end 157.829 114.975) (width 0.2) (layer Bottom) (net 60))
+  (segment (start 158.604 117.6) (end 158.604 115.75) (width 0.2) (layer Bottom) (net 60))
+  (via (at 155.725 114.8) (size 0.508) (drill 0.254) (layers Top Bottom) (net 60))
+  (segment (start 157.829 114.975) (end 155.9 114.975) (width 0.2) (layer Bottom) (net 60))
+  (segment (start 155.9 114.975) (end 155.725 114.8) (width 0.2) (layer Bottom) (net 60))
   (segment (start 155.725 110.625) (end 155.6 110.5) (width 0.2) (layer Top) (net 60))
   (segment (start 155.725 114.8) (end 155.725 110.625) (width 0.2) (layer Top) (net 60))
@@
   (segment (start 154.8 128) (end 154.8 124.05) (width 0.2) (layer Top) (net 94))
   (segment (start 154.8 124.05) (end 157.8 121.05) (width 0.2) (layer Top) (net 94))
+  (segment (start 157.875 124.925) (end 156.65 124.925) (width 0.2) (layer Bottom) (net 95))
+  (segment (start 158.604 122.4) (end 158.604 124.196) (width 0.2) (layer Bottom) (net 95))
+  (segment (start 158.604 124.196) (end 157.875 124.925) (width 0.2) (layer Bottom) (net 95))
   (via (at 155.65 125.1) (size 0.508) (drill 0.254) (layers Top Bottom) (net 95))
   (segment (start 155.65 127.95) (end 155.6 128) (width 0.2) (layer Top) (net 95))
@@
     (polygon
       (pts
-        (xy 129.2125 37.725) (xy 171.71875 37.4375) (xy 171.83125 131.7125) (xy 129.325 132)
+        (xy 129.2125 37.725) (xy 171.71875 37.4375) (xy 172 130) (xy 129.24375 130.0375)
       )
     )

Commit message: V3 of PCB hardware
3.3 to 5V level shifter added
Added decoupling caps to 5V rail and HV rail
Added cap to RESET line
Fixed locating holes in FX6 footprint
Fixed unintentional trace overlap
Eliminated the "GND" feature, and re-assigned all lines to be the common electrode
Fixed a routing error on the segment PCB, and re-assigned one common electrode line to be a segment line.
The above changes mean that the common electrode mask in firmware *must* be updated.
Parts:
- removed 3V3, SWC, SWD: TestPoint, TestPoint:TestPoint_Pad_D1.0mm
- added C10: 10n, DSKY_driver:0603-NO, F.Cu at (151.5, 99.7)
- added C11: 1uF, DSKY_driver:0603-NO, F.Cu at (133.1, 88.5)
- added C12: 1uF, DSKY_driver:0603-NO, F.Cu at (133.2, 120.8)
- added C13: 1uF, DSKY_driver:0603-NO, F.Cu at (132.7, 50.3)
- added C14: 1uF, DSKY_driver:0603-NO, F.Cu at (135.2, 111.5)
- added C15: .22u, Capacitor_SMD:C_1210_3225Metric, F.Cu at (133.7, 78.5)
- added C16: .22u, Capacitor_SMD:C_1210_3225Metric, F.Cu at (132.7, 127.5)
- added C17: .22u, Capacitor_SMD:C_1210_3225Metric, F.Cu at (132.4, 40.4)
- added LE: TestPoint, TestPoint:TestPoint_Pad_D1.0mm, F.Cu at (130.8, 123.2)
- added LOGO1: Logo_Open_Hardware_Small, Symbol:OSHW-Logo_5.7x6mm_SilkScreen, F.Cu at (168.5, 125.6)
- added MOSI: TestPoint, TestPoint:TestPoint_Pad_D1.0mm, F.Cu at (130.9, 112.9)
- added SCK: TestPoint, TestPoint:TestPoint_Pad_D1.0mm, F.Cu at (130.9, 119.7)
- added U8: CD40109B, Package_SO:TSSOP-16_4.4x5mm_P0.65mm, F.Cu at (133.2, 107.7)
- D1, D2: footprint Diode_SMD:D_SOD-123 -> DSKY_driver:D_SOD-123
- moved GND 19.2 mm to (133.3, 115.1)
- moved C1 6.53 mm to (157.8, 61.1), turned to 0 degrees
- moved R2 1.97 mm to (134.9, 102.9), turned to 180 degrees
- moved C6 1.90 mm to (134.9, 99.8)
- moved R3 1.82 mm to (134.9, 101.3)
- moved R1 0.16 mm to (142.0, 107.8)
- moved D2 0.15 mm to (140.8, 72.7), turned to 180 degrees
- moved D1 0.10 mm to (140.4, 65.2), turned to 180 degrees
Connections:
- net /D2_A1_PA09_SCL_MISO renamed Net-(IC3-Pad12)
- D1 pad 1: GND -> Net-(D1-Pad1)
- D1 pad 2: Net-(D1-Pad2) -> GND
- D2 pad 1: GND -> Net-(D2-Pad1)
- D2 pad 2: Net-(D2-Pad2) -> GND
- IC3 pad 11: /D0_A4_PA08_SDA -> Net-(IC3-Pad11)
- IC3 pad 7: /D4_A2_PA06_TXD_MOSI -> Net-(IC3-Pad7)
- IC3 pad 8: /D3_A3_PA07_RXD_SCK -> Net-(IC3-Pad8)
- J1 pad 23: GND -> (no net)
- J1 pad 24: GND -> (no net)
- J1 pad 25: GND -> (no net)
- TR1 pad 1: Net-(D1-Pad2) -> Net-(D1-Pad1)
- TR2 pad 1: Net-(D2-Pad2) -> Net-(D2-Pad1)
- U2 pad 1: Net-(D1-Pad2) -> Net-(D1-Pad1)
- U6 pad 1: Net-(D2-Pad2) -> Net-(D2-Pad1)
Routing:
- net (no net): track 0.00 -> 23.0 mm, vias 0 -> 3
- net GND: track 102.2 -> 123.0 mm, vias 41 -> 49
- net 3.3V: track 67.2 -> 81.2 mm, vias 4 -> 8
- net Net-(U7-Pad17): track 0.00 -> 9.04 mm, vias 0 -> 1
- net Net-(U7-Pad19): track 0.00 -> 9.03 mm, vias 0 -> 1
- net Net-(U7-Pad18): track 0.00 -> 9.01 mm, vias 0 -> 1
- net Net-(U5-Pad1): track 8.96 -> 0.00 mm, vias 1 -> 0
- net Net-(IC3-Pad7): track 0.00 -> 8.78 mm
- net Net-(U5-Pad64): track 7.34 -> 0.00 mm, vias 1 -> 0
- net Net-(IC3-Pad32): track 7.00 -> 0.00 mm
- net Net-(U5-Pad65): track 6.66 -> 0.00 mm, vias 1 -> 0
- net Net-(IC3-Pad11): track 0.00 -> 5.91 mm
- net Net-(D2-Pad2): track 5.56 -> 0.00 mm
- net Net-(D2-Pad1): track 0.00 -> 5.56 mm
- net /5.0V: track 147.9 -> 153.4 mm, vias 4 -> 5
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Other:
- board text added: "042119"
- board text added: "1.3A max"
- board text added: "100K"
- board text added: "10M"
- board text added: "24"
- board text added: "25"
- board text added: "40"
- board text added: "41"
- board text added: "5V"
- board text added: "64"
- board text added: "DNP"
- board text added: "DSKY_V3_DRV"
- board text added: "LSB"
- board text added: "MSB"
- board text added: "OUT1"
- board text added: "SNGL CLK = RST DBL CLK = PROG"
- board text removed: "040619"
- board text removed: "1A max"
- board text removed: "5V0"
- board text removed: "DSKY_V2_DRV"
- board text removed: "RST / PRG"
