File: PCB - KiCad/DSKY_driver/DSKY_driver.sch (KiCad schematic (older format))
At the start: 39 parts, among them IC3 ATSAMD21E, J1 Conn_15X4, J2 Conn_15X4, J3 CUI_power_jack, J4 Conn_15X4, Q2 reset, U1 HV507, U2 LT3468, U3 AP2204K-3.3, U4 AP2204K-5.0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

Commit message: V3 of PCB hardware
3.3 to 5V level shifter added
Added decoupling caps to 5V rail and HV rail
Added cap to RESET line
Fixed locating holes in FX6 footprint
Fixed unintentional trace overlap
Eliminated the "GND" feature, and re-assigned all lines to be the common electrode
Fixed a routing error on the segment PCB, and re-assigned one common electrode line to be a segment line.
The above changes mean that the common electrode mask in firmware *must* be updated.
Parts:
- removed TP1, TP2, TP3, TP4: TestPoint, TestPoint:TestPoint_Pad_D1.0mm, symbol Connector:TestPoint
- added C10: 10n, DSKY_driver:0603-NO, symbol DSKY_driver:CAP_CERAMIC0603_NO-Trinket_M0_rev_D
- added C11, C12, C13, C14: 1uF, DSKY_driver:0603-NO, symbol DSKY_driver:CAP_CERAMIC0603_NO-Trinket_M0_rev_D
- added C15, C16, C17: .22u, Capacitor_SMD:C_1210_3225Metric, symbol DSKY_driver:CAP_CERAMIC0603_NO-Trinket_M0_rev_D
- added LE1, MOSI1, MOSI2, SCK1: TestPoint, TestPoint:TestPoint_Pad_D1.0mm, symbol Connector:TestPoint
- added LOGO1: Logo_Open_Hardware_Small, Symbol:OSHW-Logo_5.7x6mm_SilkScreen, symbol Graphic:Logo_Open_Hardware_Small
- added U8: CD40109B, Package_SO:TSSOP-16_4.4x5mm_P0.65mm, symbol DSKY_driver:CD40109B
- C7, C8: value 10uF -> 2.2u
- D1, D2: footprint Diode_SMD:D_SOD-123 -> DSKY_driver:D_SOD-123; symbol pspice:DIODE -> Device:D_Schottky
Connections:
- net labels removed: D2_A1_PA09_SCL_MISO
- wire segments 245 -> 299
Other:
- moved on the sheet: C2, C6, L1, R1, R2, R3
